File: nv-h5b.brd (EAGLE design)
At the start: 8 x 20 mm, 17 parts, among them IC1 TINY13A-20SSU, J1 22-05-7038-03

Commit message: Increase main capacitor.
Parts:
- C1: value 100n -> 1u
Changed lines of the file:
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@@
 </autorouter>
 <elements>
-<element name="C1" library="rcl" package="C0805" value="100n" x="2.2225" y="6.0325" smashed="yes" rot="R180">
+<element name="C1" library="rcl" package="C0805" value="1u" x="2.2225" y="6.0325" smashed="yes" rot="R180">
 <attribute name="NAME" x="1.905" y="6.6675" size="0.8128" layer="25" rot="R270"/>
 <attribute name="VALUE" x="2.8575" y="5.08" size="0.8128" layer="27" rot="R180"/>

Commit message: Increase LED resistors (~ max. 3 mA/ LED).
Parts:
- RG, RR, RW, RYB, RYT: value 1k -> 4k7
Changed lines of the file:
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@@
 <attribute name="VALUE" x="2.42" y="6.985" size="0.0254" layer="28" rot="MR0"/>
 </element>
-<element name="RR" library="rcl" package="R0805" value="1k" x="1.905" y="18.0975" smashed="yes" rot="R270">
+<element name="RR" library="rcl" package="R0805" value="4k7" x="1.905" y="18.0975" smashed="yes" rot="R270">
 <attribute name="NAME" x="0.3175" y="18.7325" size="0.8128" layer="25" rot="R270"/>
 <attribute name="VALUE" x="0.3175" y="18.7325" size="0.8128" layer="27" rot="R270"/>
 </element>
-<element name="RG" library="rcl" package="R0805" value="1k" x="4.445" y="18.0975" smashed="yes" rot="R270">
+<element name="RG" library="rcl" package="R0805" value="4k7" x="4.445" y="18.0975" smashed="yes" rot="R270">
 <attribute name="NAME" x="2.8575" y="18.7325" size="0.8128" layer="25" rot="R270"/>
 <attribute name="VALUE" x="2.8575" y="18.7325" size="0.8128" layer="27" rot="R270"/>
 </element>
-<element name="RYT" library="rcl" package="R0805" value="1k" x="6.985" y="18.0975" smashed="yes" rot="R270">
+<element name="RYT" library="rcl" package="R0805" value="4k7" x="6.985" y="18.0975" smashed="yes" rot="R270">
 <attribute name="NAME" x="5.3975" y="19.05" size="0.8128" layer="25" rot="R270"/>
 <attribute name="VALUE" x="5.3975" y="18.7325" size="0.8128" layer="27" rot="R270"/>
 </element>
-<element name="RYB" library="rcl" package="R0805" value="1k" x="1.5875" y="13.6525" smashed="yes" rot="R270">
+<element name="RYB" library="rcl" package="R0805" value="4k7" x="1.5875" y="13.6525" smashed="yes" rot="R270">
 <attribute name="NAME" x="0.3175" y="15.24" size="0.8128" layer="25"/>
 <attribute name="VALUE" x="0" y="14.2875" size="0.8128" layer="27" rot="R270"/>
 </element>
-<element name="RW" library="rcl" package="R0805" value="1k" x="6.35" y="7.9375" smashed="yes" rot="R180">
+<element name="RW" library="rcl" package="R0805" value="4k7" x="6.35" y="7.9375" smashed="yes" rot="R180">
 <attribute name="NAME" x="4.1275" y="8.89" size="0.8128" layer="25" rot="R270"/>
 <attribute name="VALUE" x="5.08" y="8.255" size="0.8128" layer="27" rot="R180"/>
